File: hardware/master_controller/Master_Controller.kicad_pcb (KiCad board)
At the start: 4 copper layers, 140 x 95 mm, 6 parts, among them U1 STM32G474RET6, U2 LTC6820_isoSPI, U4 TCAN1042_CAN1_VCU, U5 TCAN1042_CAN2_IVTS, U6 TCAN1042_CAN3_OBC, U7 TPS274C120_Contactors

Commit message: Generate 100% complete production 4-layer PCBs with real footprints, pads, copper traces, isolation slots, and JLCPCB Gerbers
Parts:
- added C1: 100nF, C_0805_2012Metric, F.Cu at (65.0, 52.0)
- added C10: 18pF, C_0603_1608Metric, F.Cu at (60.0, 62.0)
- added C11: 100nF, C_0805_2012Metric, F.Cu at (38.0, 29.0)
- added C12: 100nF, C_0805_2012Metric, F.Cu at (38.0, 54.0)
- added C13: 100nF, C_0805_2012Metric, F.Cu at (38.0, 79.0)
- added C2: 100nF, C_0805_2012Metric, F.Cu at (85.0, 52.0)
- added C3: 100nF, C_0805_2012Metric, F.Cu at (65.0, 68.0)
- added C4: 100nF, C_0805_2012Metric, F.Cu at (85.0, 68.0)
- added C5: 100nF, C_0805_2012Metric, F.Cu at (75.0, 48.0)
- added C6: 100nF, C_0805_2012Metric, F.Cu at (75.0, 72.0)
- added C9: 18pF, C_0603_1608Metric, F.Cu at (60.0, 58.0)
- added D1: SMBJ36CA_TVS, D_SMB, F.Cu at (40.0, 20.0)
- added D2: 1000V_1A_Flyback, D_SMA, F.Cu at (100.0, 90.0)
- added D3: 1000V_1A_Flyback, D_SMA, F.Cu at (115.0, 90.0)
- added D4: 1000V_1A_Flyback, D_SMA, F.Cu at (130.0, 90.0)
- added D5: 1000V_1A_Flyback, D_SMA, F.Cu at (145.0, 90.0)
- added D6: TVS_CAN, D_SMA, F.Cu at (25.0, 41.0)
- added D7: TVS_CAN, D_SMA, F.Cu at (25.0, 66.0)
- added D8: TVS_CAN, D_SMA, F.Cu at (25.0, 91.0)
- added H1: M3, MountingHole_3.2mm_M3, F.Cu at (16.0, 16.0)
- added H2: M3, MountingHole_3.2mm_M3, F.Cu at (154.0, 16.0)
- added H3: M3, MountingHole_3.2mm_M3, F.Cu at (16.0, 104.0)
- added H4: M3, MountingHole_3.2mm_M3, F.Cu at (154.0, 104.0)
- added J1: Contactor_Outputs_8P, Molex_Mini-Fit_Jr_5566-08A_2x04_P4.20mm_Vertical, F.Cu at (125.0, 102.0)
- added J2: CAN_Harness_12P, Molex_Micro-Fit_3.0_43045-1200_2x06_P3.00mm_Horizontal, F.Cu at (16.0, 60.0)
- added J3: isoSPI_PortA, Molex_Micro-Fit_3.0_43045-0400_2x02_P3.00mm_Horizontal, F.Cu at (152.0, 30.0)
- added J4: isoSPI_PortB, Molex_Micro-Fit_3.0_43045-0400_2x02_P3.00mm_Horizontal, F.Cu at (152.0, 50.0)
- added R1: 1M0_500V, R_1206_3216Metric, F.Cu at (50.0, 100.0)
- added R2: 1M0_500V, R_1206_3216Metric, F.Cu at (58.0, 100.0)
- added R3: 1M0_500V, R_1206_3216Metric, F.Cu at (70.0, 100.0)
- added R4: 1M0_500V, R_1206_3216Metric, F.Cu at (78.0, 100.0)
- added R5: 120R, R_0805_2012Metric, F.Cu at (22.0, 35.0)
- added R6: 120R, R_0805_2012Metric, F.Cu at (22.0, 60.0)
- added R7: 120R, R_0805_2012Metric, F.Cu at (22.0, 85.0)
- added T1: HM2101NL_PortA, SOIC-16_3.9x9.9mm_P1.27mm, F.Cu at (125.0, 30.0)
- added T2: HM2101NL_PortB, SOIC-16_3.9x9.9mm_P1.27mm, F.Cu at (125.0, 50.0)
- added U10: TPS274C_PWM_Fan, SOIC-8_3.9x4.9mm_P1.27mm, F.Cu at (145.0, 80.0)
- added U11: VO14642_IMD_Pos, SOIC-8_3.9x4.9mm_P1.27mm, F.Cu at (55.0, 90.0)
- added U12: VO14642_IMD_Neg, SOIC-8_3.9x4.9mm_P1.27mm, F.Cu at (75.0, 90.0)
- added U13: LM5164_12V_Buck, SOIC-8_3.9x4.9mm_P1.27mm, F.Cu at (50.0, 30.0)
- added U14: TLV70233_LDO, SOT-23, F.Cu at (65.0, 30.0)
- added U3: LTC6820_PortB, SOIC-16_3.9x9.9mm_P1.27mm, F.Cu at (100.0, 50.0)
- added U8: TPS274C_MainNeg, SOIC-8_3.9x4.9mm_P1.27mm, F.Cu at (115.0, 80.0)
- added U9: TPS274C_Precharge, SOIC-8_3.9x4.9mm_P1.27mm, F.Cu at (130.0, 80.0)
- added Y1: 8.000MHz, Crystal_SMD_3225-4Pin_3.2x2.5mm, F.Cu at (65.0, 60.0)
- U1: footprint Package_QFP:LQFP-64_10x10mm_P0.5mm -> LQFP-64_10x10mm_P0.5mm
- U2: value LTC6820_isoSPI -> LTC6820_PortA; footprint Package_SO:MSOP-16_3x4mm_P0.5mm -> SOIC-16_3.9x9.9mm_P1.27mm
- U4: value TCAN1042_CAN1_VCU -> TCAN1042_CAN1_Vehicle; footprint Package_SO:SOIC-8_3.9x4.9mm_P1.27mm -> SOIC-8_3.9x4.9mm_P1.27mm
- U5: footprint Package_SO:SOIC-8_3.9x4.9mm_P1.27mm -> SOIC-8_3.9x4.9mm_P1.27mm
- U6: value TCAN1042_CAN3_OBC -> TCAN1042_CAN3_Charger; footprint Package_SO:SOIC-8_3.9x4.9mm_P1.27mm -> SOIC-8_3.9x4.9mm_P1.27mm
- U7: value TPS274C120_Contactors -> TPS274C_MainPos; footprint Package_DFN_QFN:WQFN-16-1EP_4x4mm_P0.5mm_EP2.6x2.6mm -> SOIC-8_3.9x4.9mm_P1.27mm
- moved U2 62.6 mm to (100.0, 30.0)
- moved U7 42.4 mm to (100.0, 80.0)
- moved U4 14.1 mm to (30.0, 35.0)
- moved U1 11.2 mm to (75.0, 60.0)
- moved U5 11.2 mm to (30.0, 60.0)
- moved U6 10.0 mm to (30.0, 85.0)
Routing:
- net +3.3V: track 0.00 -> 136.0 mm
- net GND: track 0.00 -> 130.9 mm
- net SPI1_SCK: track 0.00 -> 113.1 mm
- net SPI2_CS_B: track 0.00 -> 80.4 mm
- net CAN3_L: track 0.00 -> 51.1 mm
- net CAN1_L: track 0.00 -> 45.6 mm
- net DRV_FAN_PWM: track 0.00 -> 23.0 mm
- net ISOSPI_B_P: track 0.00 -> 22.0 mm
- net ISOSPI_B_N: track 0.00 -> 22.0 mm
- net ISOSPI_A_P: track 0.00 -> 22.0 mm
- net ISOSPI_A_N: track 0.00 -> 22.0 mm
- net DRV_MAIN_POS: track 0.00 -> 21.2 mm
- net DRV_PRECHARGE: track 0.00 -> 16.4 mm
- net DRV_MAIN_NEG: track 0.00 -> 15.6 mm
- net +12V_KL30: track 0.00 -> 11.3 mm
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Other:
- board size 140 x 95 mm -> 150 x 100 mm
- copper layers 4 -> 2
- rule pad_to_mask_clearance: 0.05 -> 0
- board text added: "CAN HARNESS (J2)"
- board text added: "CONTACTOR OUTPUTS (J1)"
- board text added: "ISOLATION MOAT (4300Vdc)"
- board text added: "OpenEV-BMS MASTER CONTROLLER v1.0"
- board text added: "STM32G474 + Triple CAN + IVT-S + IMD"
- board text added: "isoSPI A"
- board text added: "isoSPI B"
- board text removed: "OpenEV-BMS Master Controller (STM32G474 + Triple CAN + IMD)"
