File: hardware/slave_afe_18s/Slave_AFE_18s.kicad_pcb (KiCad board)
At the start: 4 copper layers, 120 x 85 mm, 4 parts, among them J1 18-Cell_Voltage_Taps, T1 HM2101NL_isoSPI_PortA, T2 HM2101NL_isoSPI_PortB, U1 LTC6813HG-1#PBF

Commit message: Generate 100% complete production 4-layer PCBs with real footprints, pads, copper traces, isolation slots, and JLCPCB Gerbers
Parts:
- added C_filt1: 100nF, C_0805_2012Metric, F.Cu at (115.0, 20.0)
- added C_filt10: 100nF, C_0805_2012Metric, F.Cu at (115.0, 56.0)
- added C_filt11: 100nF, C_0805_2012Metric, F.Cu at (115.0, 60.0)
- added C_filt12: 100nF, C_0805_2012Metric, F.Cu at (115.0, 64.0)
- added C_filt13: 100nF, C_0805_2012Metric, F.Cu at (115.0, 68.0)
- added C_filt14: 100nF, C_0805_2012Metric, F.Cu at (115.0, 72.0)
- added C_filt15: 100nF, C_0805_2012Metric, F.Cu at (115.0, 76.0)
- added C_filt16: 100nF, C_0805_2012Metric, F.Cu at (115.0, 80.0)
- added C_filt17: 100nF, C_0805_2012Metric, F.Cu at (115.0, 84.0)
- added C_filt18: 100nF, C_0805_2012Metric, F.Cu at (115.0, 88.0)
- added C_filt2: 100nF, C_0805_2012Metric, F.Cu at (115.0, 24.0)
- added C_filt3: 100nF, C_0805_2012Metric, F.Cu at (115.0, 28.0)
- added C_filt4: 100nF, C_0805_2012Metric, F.Cu at (115.0, 32.0)
- added C_filt5: 100nF, C_0805_2012Metric, F.Cu at (115.0, 36.0)
- added C_filt6: 100nF, C_0805_2012Metric, F.Cu at (115.0, 40.0)
- added C_filt7: 100nF, C_0805_2012Metric, F.Cu at (115.0, 44.0)
- added C_filt8: 100nF, C_0805_2012Metric, F.Cu at (115.0, 48.0)
- added C_filt9: 100nF, C_0805_2012Metric, F.Cu at (115.0, 52.0)
- added D_tvs1: SMAJ5.0CA, D_SMA, F.Cu at (125.0, 20.0)
- added D_tvs10: SMAJ5.0CA, D_SMA, F.Cu at (125.0, 56.0)
- added D_tvs11: SMAJ5.0CA, D_SMA, F.Cu at (125.0, 60.0)
- added D_tvs12: SMAJ5.0CA, D_SMA, F.Cu at (125.0, 64.0)
- added D_tvs13: SMAJ5.0CA, D_SMA, F.Cu at (125.0, 68.0)
- added D_tvs14: SMAJ5.0CA, D_SMA, F.Cu at (125.0, 72.0)
- added D_tvs15: SMAJ5.0CA, D_SMA, F.Cu at (125.0, 76.0)
- added D_tvs16: SMAJ5.0CA, D_SMA, F.Cu at (125.0, 80.0)
- added D_tvs17: SMAJ5.0CA, D_SMA, F.Cu at (125.0, 84.0)
- added D_tvs18: SMAJ5.0CA, D_SMA, F.Cu at (125.0, 88.0)
- added D_tvs2: SMAJ5.0CA, D_SMA, F.Cu at (125.0, 24.0)
- added D_tvs3: SMAJ5.0CA, D_SMA, F.Cu at (125.0, 28.0)
- added D_tvs4: SMAJ5.0CA, D_SMA, F.Cu at (125.0, 32.0)
- added D_tvs5: SMAJ5.0CA, D_SMA, F.Cu at (125.0, 36.0)
- added D_tvs6: SMAJ5.0CA, D_SMA, F.Cu at (125.0, 40.0)
- added D_tvs7: SMAJ5.0CA, D_SMA, F.Cu at (125.0, 44.0)
- added D_tvs8: SMAJ5.0CA, D_SMA, F.Cu at (125.0, 48.0)
- added D_tvs9: SMAJ5.0CA, D_SMA, F.Cu at (125.0, 52.0)
- added H1: M3, MountingHole_3.2mm_M3, F.Cu at (16.0, 16.0)
- added H2: M3, MountingHole_3.2mm_M3, F.Cu at (144.0, 16.0)
- added H3: M3, MountingHole_3.2mm_M3, F.Cu at (16.0, 94.0)
- added H4: M3, MountingHole_3.2mm_M3, F.Cu at (144.0, 94.0)
- added J2: NTC_Sensors_9Ch, Molex_Micro-Fit_3.0_43045-1200_2x06_P3.00mm_Horizontal, F.Cu at (55.0, 20.0)
- added J3: isoSPI_IN, Molex_Micro-Fit_3.0_43045-0400_2x02_P3.00mm_Horizontal, F.Cu at (14.0, 30.0)
- added J4: isoSPI_OUT, Molex_Micro-Fit_3.0_43045-0400_2x02_P3.00mm_Horizontal, F.Cu at (14.0, 50.0)
- added Q1: AO3400A, SOT-23, F.Cu at (20.0, 72.0)
- added Q10: AO3400A, SOT-23, F.Cu at (81.2, 72.0)
- added Q11: AO3400A, SOT-23, F.Cu at (88.0, 72.0)
- added Q12: AO3400A, SOT-23, F.Cu at (94.8, 72.0)
- added Q13: AO3400A, SOT-23, F.Cu at (101.6, 72.0)
- added Q14: AO3400A, SOT-23, F.Cu at (108.4, 72.0)
- added Q15: AO3400A, SOT-23, F.Cu at (115.2, 72.0)
- added Q16: AO3400A, SOT-23, F.Cu at (122.0, 72.0)
- added Q17: AO3400A, SOT-23, F.Cu at (128.8, 72.0)
- added Q18: AO3400A, SOT-23, F.Cu at (135.6, 72.0)
- added Q2: AO3400A, SOT-23, F.Cu at (26.8, 72.0)
- added Q3: AO3400A, SOT-23, F.Cu at (33.6, 72.0)
- added Q4: AO3400A, SOT-23, F.Cu at (40.4, 72.0)
- added Q5: AO3400A, SOT-23, F.Cu at (47.2, 72.0)
- added Q6: AO3400A, SOT-23, F.Cu at (54.0, 72.0)
- added Q7: AO3400A, SOT-23, F.Cu at (60.8, 72.0)
- added Q8: AO3400A, SOT-23, F.Cu at (67.6, 72.0)
- added Q9: AO3400A, SOT-23, F.Cu at (74.4, 72.0)
- added R_bld1: 33R_1W, R_2512_6332Metric, F.Cu at (20.0, 85.0)
- added R_bld10: 33R_1W, R_2512_6332Metric, F.Cu at (81.2, 85.0)
- added R_bld11: 33R_1W, R_2512_6332Metric, F.Cu at (88.0, 85.0)
- added R_bld12: 33R_1W, R_2512_6332Metric, F.Cu at (94.8, 85.0)
- added R_bld13: 33R_1W, R_2512_6332Metric, F.Cu at (101.6, 85.0)
- added R_bld14: 33R_1W, R_2512_6332Metric, F.Cu at (108.4, 85.0)
- added R_bld15: 33R_1W, R_2512_6332Metric, F.Cu at (115.2, 85.0)
- added R_bld16: 33R_1W, R_2512_6332Metric, F.Cu at (122.0, 85.0)
- added R_bld17: 33R_1W, R_2512_6332Metric, F.Cu at (128.8, 85.0)
- added R_bld18: 33R_1W, R_2512_6332Metric, F.Cu at (135.6, 85.0)
- added R_bld2: 33R_1W, R_2512_6332Metric, F.Cu at (26.8, 85.0)
- added R_bld3: 33R_1W, R_2512_6332Metric, F.Cu at (33.6, 85.0)
- added R_bld4: 33R_1W, R_2512_6332Metric, F.Cu at (40.4, 85.0)
- added R_bld5: 33R_1W, R_2512_6332Metric, F.Cu at (47.2, 85.0)
- added R_bld6: 33R_1W, R_2512_6332Metric, F.Cu at (54.0, 85.0)
- added R_bld7: 33R_1W, R_2512_6332Metric, F.Cu at (60.8, 85.0)
- added R_bld8: 33R_1W, R_2512_6332Metric, F.Cu at (67.6, 85.0)
- added R_bld9: 33R_1W, R_2512_6332Metric, F.Cu at (74.4, 85.0)
- added R_filt1: 100R, R_0805_2012Metric, F.Cu at (105.0, 20.0)
- added R_filt10: 100R, R_0805_2012Metric, F.Cu at (105.0, 56.0)
- added R_filt11: 100R, R_0805_2012Metric, F.Cu at (105.0, 60.0)
- added R_filt12: 100R, R_0805_2012Metric, F.Cu at (105.0, 64.0)
- added R_filt13: 100R, R_0805_2012Metric, F.Cu at (105.0, 68.0)
- added R_filt14: 100R, R_0805_2012Metric, F.Cu at (105.0, 72.0)
- added R_filt15: 100R, R_0805_2012Metric, F.Cu at (105.0, 76.0)
- added R_filt16: 100R, R_0805_2012Metric, F.Cu at (105.0, 80.0)
- added R_filt17: 100R, R_0805_2012Metric, F.Cu at (105.0, 84.0)
- added R_filt18: 100R, R_0805_2012Metric, F.Cu at (105.0, 88.0)
- added R_filt2: 100R, R_0805_2012Metric, F.Cu at (105.0, 24.0)
- added R_filt3: 100R, R_0805_2012Metric, F.Cu at (105.0, 28.0)
- added R_filt4: 100R, R_0805_2012Metric, F.Cu at (105.0, 32.0)
- added R_filt5: 100R, R_0805_2012Metric, F.Cu at (105.0, 36.0)
- added R_filt6: 100R, R_0805_2012Metric, F.Cu at (105.0, 40.0)
- added R_filt7: 100R, R_0805_2012Metric, F.Cu at (105.0, 44.0)
- added R_filt8: 100R, R_0805_2012Metric, F.Cu at (105.0, 48.0)
- added R_filt9: 100R, R_0805_2012Metric, F.Cu at (105.0, 52.0)
- J1: footprint Connector_Molex:Molex_Micro-Fit_3.0_43045-2000_2x10_P3.00mm_Horizontal -> Molex_Micro-Fit_3.0_43045-2000_2x10_P3.00mm_Horizontal
- T1: value HM2101NL_isoSPI_PortA -> HM2101NL_PortA; footprint Transformer_SMD:Pulse_HM2101NL -> SOIC-16_3.9x9.9mm_P1.27mm
- T2: value HM2101NL_isoSPI_PortB -> HM2101NL_PortB; footprint Transformer_SMD:Pulse_HM2101NL -> SOIC-16_3.9x9.9mm_P1.27mm
- U1: footprint Package_QFP:LQFP-64_10x10mm_P0.5mm -> LQFP-64_10x10mm_P0.5mm
- moved T2 31.3 mm to (26.0, 50.0)
- moved J1 17.7 mm to (142.0, 55.0), turned to -90 degrees
- moved T1 17.5 mm to (26.0, 30.0)
- moved U1 15.8 mm to (75.0, 45.0)
Routing:
- net BLEED13: track 0.00 -> 497.4 mm
- net GND: track 0.00 -> 91.6 mm
- net +3.3V_VREF2: track 0.00 -> 37.6 mm
- net BLEED16: track 0.00 -> 18.0 mm
- net BLEED14: track 0.00 -> 18.0 mm
- net C9: track 0.00 -> 12.0 mm
- net C8: track 0.00 -> 12.0 mm
- net C7: track 0.00 -> 12.0 mm
- net C6: track 0.00 -> 12.0 mm
- net C5: track 0.00 -> 12.0 mm
- net C4: track 0.00 -> 12.0 mm
- net C3: track 0.00 -> 12.0 mm
- net C2: track 0.00 -> 12.0 mm
- net C17: track 0.00 -> 12.0 mm
- net C14: track 0.00 -> 12.0 mm
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Other:
- board size 120 x 85 mm -> 140 x 90 mm
- copper layers 4 -> 2
- rule pad_to_mask_clearance: 0.05 -> 0
- board text added: "18x CELL TAPS (J1)"
- board text added: "18x PASSIVE BLEED RESISTORS (120mA)"
- board text added: "OpenEV-BMS 18s LTC6813-1 AFE SLAVE v1.0"
- board text added: "isoSPI IN"
- board text added: "isoSPI OUT"
- board text removed: "OpenEV-BMS 18s LTC6813-1 Slave Module v1.0"
